File: borsdorf.kicad_pcb (KiCad board)
At the start: 2 copper layers, 314.3 x 95.2 mm, 162 parts, among them J1 USB-2.0_USB-C, K1 KEYSW, K10 KEYSW, K11 KEYSW, K12 KEYSW, K13 KEYSW, K14 KEYSW, K15 KEYSW, K16 KEYSW, K17 KEYSW, K18 KEYSW, K19 KEYSW, K2 KEYSW, K20 KEYSW, K21 KEYSW, K22 KEYSW, K23 KEYSW, K24 KEYSW, K25 KEYSW, K26 KEYSW, K27 KEYSW, K28 KEYSW, K29 KEYSW, K3 KEYSW, K30 KEYSW, K31 KEYSW, K32 KEYSW, K33 KEYSW, K34 KEYSW, K35 KEYSW, K36 KEYSW, K37 KEYSW, K38 KEYSW, K39 KEYSW, K4 KEYSW, K40 KEYSW, K41 KEYSW, K42 KEYSW, K43 KEYSW, K44 KEYSW, K45 KEYSW, K46 KEYSW, K47 KEYSW, K48 KEYSW, K49 KEYSW, K5 KEYSW, K50 KEYSW, K51 KEYSW, K52 KEYSW, K53 KEYSW, K54 KEYSW, K55 KEYSW, K56 KEYSW, K56-2 KEYSW, K57 KEYSW, K58 KEYSW, K59 KEYSW, K6 KEYSW, K60 KEYSW, K61 KEYSW, K62 KEYSW, K63 KEYSW, K64 KEYSW, K65 KEYSW, K66 KEYSW, K67 KEYSW, K7 KEYSW, K8 KEYSW, K9 KEYSW, SW1 ALPS SKRK, SW2 ALPS SSSS811101, U1 USBLC6-2P6, U2 LP2985-3.3, U3 STM32F072CBTx

Commit message: Update to v02
Parts:
- removed D1: D_Schottky_Small_ALT, Diode_SMD:D_SOD-123
- removed the G*** at (217.0, 123.0)
- removed REF**: SerialNumber, Cutie_Club:SerialNumber
- added G***: LOGO, Cutie_Club:Borsdorf, B.Cu at (200.0, 124.0)
- added G***: LOGO, Cutie_Club:newLogoCC, B.Cu at (160.0, 124.0)
- J1: value USB-2.0_USB-C -> USB2.0-USB-C; footprint Cutie Club:TYPE-C-31-M-12 -> Connector_USB:USB_C_Receptacle_HRO_TYPE-C-31-M-12
- moved R2 3.25 mm to (328.2, 47.8)
- moved R3 3.25 mm to (325.2, 47.8)
- moved J1 0.60 mm to (326.2, 40.5)
- renumbered U3 to U1, U1 to U3
Connections:
- F1 pad 2: Net-(D1-Pad1) -> VBUS
- R2 pad 1: Net-(J1-Pad6) -> Net-(J1-PadB5)
- R3 pad 1: Net-(J1-Pad7) -> Net-(J1-PadA5)
Routing:
- net Net-(J1-Pad3): track 5.40 -> 0.00 mm
- net VBUS: track 11.6 -> 15.0 mm
- net Net-(D1-Pad1): track 3.04 -> 0.00 mm
- net Net-(J1-Pad7): track 2.51 -> 0.00 mm
- net Net-(J1-PadB5): track 0.00 -> 2.40 mm
- net Net-(J1-PadA5): track 0.00 -> 2.40 mm
- net Net-(J1-Pad6): track 2.30 -> 0.00 mm
- net COL8: track 195.7 -> 194.6 mm
- net COL14: track 148.2 -> 149.2 mm, vias 2 -> 0
- net ROW0: track 314.6 -> 315.4 mm, vias 4 -> 2
- net Cond_D+: track 29.1 -> 29.3 mm, vias 0 -> 2
- net ROW1: track 286.0 -> 285.9 mm, vias 2 -> 0
- net Cond_D-: vias 0 -> 2
Other:
- outline, holes or cut-outs redrawn
- net class Default: clearance 0.127 -> 0.1
- rule pad_to_mask_clearance: 0.0508 -> 0
- rule trace_clearance: 0.127 -> 0.1
- board text removed: "Borsdorf Prototype"
- board text removed: "JLCJLCJLCJLC"

Commit message: Update Borsdorf to production files
Parts:
- removed C13: 100nF, Capacitor_SMD:C_0805_2012Metric
- C12: value 4.7uF -> 100nF
- C2: value 100nF -> 1uF
- C3: value 100nF -> 4.7uF
- C5: value 1uF -> 100nF
- moved C2 17.1 mm to (322.0, 98.5), turned to 0 degrees
- moved C1 15.3 mm to (318.1, 86.5), turned to 0 degrees
- moved C12 13.4 mm to (329.5, 83.1), turned to 180 degrees
- moved C3 12.4 mm to (329.5, 81.1)
- moved C5 10.5 mm to (331.2, 92.7), turned to 90 degrees
- moved R4 9.09 mm to (340.6, 93.8), turned to 90 degrees
- moved C10 5.06 mm to (318.6, 56.9), turned to 0 degrees
- moved C11 4.40 mm to (315.8, 53.9), turned to -90 degrees
- moved C6 2.97 mm to (322.0, 100.5)
- moved F1 1.15 mm to (323.8, 52.1)
- moved U2 0.90 mm to (318.8, 54.0)
- moved C9 0.89 mm to (323.8, 55.9), turned to -90 degrees
- moved C4 0.81 mm to (318.1, 84.5)
- moved C8 0.77 mm to (321.8, 54.0), turned to -90 degrees
- moved C7 0.40 mm to (337.5, 93.8), turned to -90 degrees
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Connections:
- C1 pad 1: VDDA -> GND
- C1 pad 2: GND -> VDD
- C11 pad 1: VDDA -> VDD
- C12 pad 1: VDDA -> VDD
- C2 pad 1: VDDA -> VDD
- C3 pad 1: VDDA -> VDD
- C4 pad 1: VDDA -> VDD
- C5 pad 1: VDDA -> VDD
- C6 pad 1: VDDA -> VDD
- J1 pad A8: (no net) -> Net-(J1-PadA8)
- J1 pad B8: (no net) -> Net-(J1-PadB8)
- SW2 pad 1: VDDA -> VDD
- U1 pad 1: VDDA -> VDD
- U1 pad 2: (no net) -> Net-(U1-Pad2)
- U1 pad 24: VDDA -> VDD
- U1 pad 27: (no net) -> Net-(U1-Pad27)
- U1 pad 28: (no net) -> Net-(U1-Pad28)
- U1 pad 29: (no net) -> Net-(U1-Pad29)
- U1 pad 3: (no net) -> Net-(U1-Pad3)
- U1 pad 30: (no net) -> Net-(U1-Pad30)
- U1 pad 31: (no net) -> Net-(U1-Pad31)
- U1 pad 34: (no net) -> Net-(U1-Pad34)
- U1 pad 36: VDDA -> VDD
- U1 pad 39: (no net) -> Net-(U1-Pad39)
- U1 pad 4: (no net) -> Net-(U1-Pad4)
- U1 pad 42: (no net) -> Net-(U1-Pad42)
- U1 pad 43: (no net) -> Net-(U1-Pad43)
- U1 pad 45: (no net) -> Net-(U1-Pad45)
- U1 pad 46: (no net) -> Net-(U1-Pad46)
- U1 pad 48: VDDA -> VDD
- U1 pad 9: VDDA -> VDD
- U2 pad 5: VDDA -> VDD
Routing:
- net VDD: track 0.00 -> 162.9 mm, vias 0 -> 8
- net VDDA: track 119.6 -> 0.00 mm, vias 6 -> 0
- net GND: track 7.51 -> 22.0 mm
- net BOOT0: track 1.90 -> 13.2 mm, vias 0 -> 2
- net Net-(R4-Pad1): track 15.1 -> 8.91 mm, vias 2 -> 0
- net RESET: track 28.7 -> 25.3 mm
- net COL2: track 324.7 -> 327.8 mm
- net COL6: track 247.6 -> 250.7 mm
- net COL13: track 136.1 -> 138.3 mm
- net COL14: track 149.2 -> 147.3 mm
- net ROW0: track 315.4 -> 316.6 mm
- net VBUS: track 15.0 -> 13.9 mm
- net ROW4: track 306.0 -> 304.9 mm
- net ROW3: track 301.6 -> 300.5 mm
- net Net-(D15-Pad2): track 13.2 -> 14.1 mm
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Other:
- net class Default removed

Commit message: Update files to v2/extras revision
Parts:
- removed C11: 2.2uF, Capacitor_SMD:C_0805_2012Metric
- removed C12: 100nF, Capacitor_SMD:C_0805_2012Metric
- removed D10, D11, D12, D13, D14, D15, D17, D18, D19, D2, D20, D21, D22, D23, D24, D25, D26, D27, D28, D29, D3, D30, D31, D32, D33, D34, D35, D36, D37, D38, D39, D4, D40, D41, D42, D43, D44, D45, D46, D47, D48, D49, D5, D50, D51, D52, D53, D54, D55, D56, D57, D58, D59, D6, D60, D61, D62, D63, D64, D65, D66, D67, D68, D7, D8, D9: D, Diode_SMD:D_SOD-123
- removed the G*** at (160.0, 124.0)
- removed the G*** at (200.0, 124.0)
- removed K45, K56, K59: KEYSW, Cutie Club:ALPS_SKxx_19.05mm
- removed R1: R_Small, Resistor_SMD:R_0805_2012Metric
- removed R3: 5.1k, Resistor_SMD:R_0805_2012Metric
- removed SW2: ALPS SSSS811101, Button_Switch_SMD:SW_SPDT_PCM12
- added C111: 10nF, Capacitor_SMD:C_0805_2012Metric, B.Cu at (318.5, 57.0)
- added C112: 2.2uF, Capacitor_SMD:C_0805_2012Metric, B.Cu at (331.2, 92.8)
- added D101: 1N4148, Diode_SMD:D_SOD-323, B.Cu at (335.5, 98.5)
- added D102: BAV70, Package_TO_SOT_SMD:SOT-23, B.Cu at (59.5, 54.8)
- added D103: BAV70, Package_TO_SOT_SMD:SOT-23, B.Cu at (97.6, 54.8)
- added D104: BAV70, Package_TO_SOT_SMD:SOT-23, B.Cu at (135.7, 54.8)
- added D105: BAV70, Package_TO_SOT_SMD:SOT-23, B.Cu at (173.8, 54.8)
- added D106: BAV70, Package_TO_SOT_SMD:SOT-23, B.Cu at (211.9, 54.8)
- added D107: BAV70, Package_TO_SOT_SMD:SOT-23, B.Cu at (250.0, 54.8)
- added D108: BAV70, Package_TO_SOT_SMD:SOT-23, B.Cu at (290.5, 54.8)
- added D109: BAV70, Package_TO_SOT_SMD:SOT-23, B.Cu at (331.0, 54.8)
- added D110: BAV70, Package_TO_SOT_SMD:SOT-23, B.Cu at (64.3, 73.8)
- added D111: BAV70, Package_TO_SOT_SMD:SOT-23, B.Cu at (107.2, 73.8)
- added D112: BAV70, Package_TO_SOT_SMD:SOT-23, B.Cu at (145.3, 73.8)
- added D113: BAV70, Package_TO_SOT_SMD:SOT-23, B.Cu at (183.4, 73.8)
- added D114: BAV70, Package_TO_SOT_SMD:SOT-23, B.Cu at (221.5, 73.8)
- added D115: BAV70, Package_TO_SOT_SMD:SOT-23, B.Cu at (259.6, 73.8)
- added D117: BAV70, Package_TO_SOT_SMD:SOT-23, B.Cu at (66.7, 92.9)
- added D118: BAV70, Package_TO_SOT_SMD:SOT-23, B.Cu at (111.9, 92.9)
- added D119: BAV70, Package_TO_SOT_SMD:SOT-23, B.Cu at (150.0, 92.9)
- added D120: BAV70, Package_TO_SOT_SMD:SOT-23, B.Cu at (188.1, 92.9)
- added D121: BAV70, Package_TO_SOT_SMD:SOT-23, B.Cu at (226.2, 92.9)
- added D122: BAV70, Package_TO_SOT_SMD:SOT-23, B.Cu at (264.3, 92.9)
- added D123: BAV70, Package_TO_SOT_SMD:SOT-23, B.Cu at (302.4, 92.9)
- added D124: BAV70, Package_TO_SOT_SMD:SOT-23, B.Cu at (61.9, 111.9)
- added D125: BAV70, Package_TO_SOT_SMD:SOT-23, B.Cu at (102.4, 111.9)
- added D126: BAV70, Package_TO_SOT_SMD:SOT-23, B.Cu at (140.5, 111.9)
- added D127: BAV70, Package_TO_SOT_SMD:SOT-23, B.Cu at (178.6, 111.9)
- added D128: BAV70, Package_TO_SOT_SMD:SOT-23, B.Cu at (216.7, 111.9)
- added D129: BAV70, Package_TO_SOT_SMD:SOT-23, B.Cu at (254.8, 111.9)
- added D130: BAV70, Package_TO_SOT_SMD:SOT-23, B.Cu at (311.9, 111.9)
- added D131: BAV70, Package_TO_SOT_SMD:SOT-23, B.Cu at (331.0, 111.9)
- added D132: BAV70, Package_TO_SOT_SMD:SOT-23, B.Cu at (61.9, 123.8)
- added D133: BAV70, Package_TO_SOT_SMD:SOT-23, B.Cu at (114.3, 123.8)
- added D134: BAV70, Package_TO_SOT_SMD:SOT-23, B.Cu at (269.1, 123.8)
- added D135: BAV70, Package_TO_SOT_SMD:SOT-23, B.Cu at (311.9, 123.8)
- added D136: BAV70, Package_TO_SOT_SMD:SOT-23, B.Cu at (331.0, 123.8)
- added G***: LOGO, Borsdorf:ccroundel, F.Cu at (235.7, 123.8)
- added G***: LOGO, Borsdorf:ccroundel, B.Cu at (197.6, 123.8)
- added K145: KEYSW, cutie-lib-alps:Alps_SKxx_19.05mm_1.0u, F.Cu at (73.8, 104.8)
- added K1571: KEYSW, cutie-lib-alps:Alps_SKxx_19.05mm_1.0u, F.Cu at (292.9, 104.8)
- added K159: KEYSW, cutie-lib-alps:Alps_SKxx_19.05mm_1.0u, F.Cu at (50.0, 123.8)
- added Q101: MBT2222A, Package_TO_SOT_SMD:SOT-23-3, B.Cu at (335.5, 104.0)
- added QR*****: 00BRDF020101, Borsdorf:00BRDF020101, B.Cu at (165.3, 123.8)
- added R101: 5.1k, Resistor_SMD:R_0805_2012Metric, B.Cu at (325.2, 47.8)
- added R103: 30k, Resistor_SMD:R_0805_2012Metric, B.Cu at (332.0, 98.5)
- added R105: R_Small, Resistor_SMD:R_0805_2012Metric, B.Cu at (54.8, 76.0)
- C105: renamed from C5; value 100nF -> 10uF
- C106: renamed from C6; value 10nF -> 100nF
- C107: renamed from C7; value 100nF -> 10nF
- C108: renamed from C8; value 1uF -> 100nF
- C109: renamed from C9; value 100nF -> 1uF
- C110: renamed from C10; value 10nF -> 100nF
- D116: renamed from D16; value D -> BAV70; footprint Diode_SMD:D_SOD-123 -> Package_TO_SOT_SMD:SOT-23
- K101: renamed from K1; footprint Cutie Club:ALPS_SKxx_19.05mm -> cutie-lib-alps:Alps_SKxx_19.05mm_1.0u
- K102: renamed from K2; footprint Cutie Club:ALPS_SKxx_19.05mm -> cutie-lib-alps:Alps_SKxx_19.05mm_1.0u
- K103: renamed from K3; footprint Cutie Club:ALPS_SKxx_19.05mm -> cutie-lib-alps:Alps_SKxx_19.05mm_1.0u
- K104: renamed from K4; footprint Cutie Club:ALPS_SKxx_19.05mm -> cutie-lib-alps:Alps_SKxx_19.05mm_1.0u
- K105: renamed from K5; footprint Cutie Club:ALPS_SKxx_19.05mm -> cutie-lib-alps:Alps_SKxx_19.05mm_1.0u
- K106: renamed from K6; footprint Cutie Club:ALPS_SKxx_19.05mm -> cutie-lib-alps:Alps_SKxx_19.05mm_1.0u
- K107: renamed from K7; footprint Cutie Club:ALPS_SKxx_19.05mm -> cutie-lib-alps:Alps_SKxx_19.05mm_1.0u
- K108: renamed from K8; footprint Cutie Club:ALPS_SKxx_19.05mm -> cutie-lib-alps:Alps_SKxx_19.05mm_1.0u
- K109: renamed from K9; footprint Cutie Club:ALPS_SKxx_19.05mm -> cutie-lib-alps:Alps_SKxx_19.05mm_1.0u
- K110: renamed from K10; footprint Cutie Club:ALPS_SKxx_19.05mm -> cutie-lib-alps:Alps_SKxx_19.05mm_1.0u
- K111: renamed from K11; footprint Cutie Club:ALPS_SKxx_19.05mm -> cutie-lib-alps:Alps_SKxx_19.05mm_1.0u
- K112: renamed from K12; footprint Cutie Club:ALPS_SKxx_19.05mm -> cutie-lib-alps:Alps_SKxx_19.05mm_1.0u
- K113: renamed from K13; footprint Cutie Club:ALPS_SKxx_19.05mm -> cutie-lib-alps:Alps_SKxx_19.05mm_1.0u
- K114: renamed from K14; footprint Cutie Club:ALPS_SKxx_19.05mm -> cutie-lib-alps:Alps_SKxx_19.05mm_1.0u
- K115: renamed from K15; footprint Cutie Club:ALPS_SKxx_19.05mm -> cutie-lib-alps:Alps_SKxx_19.05mm_1.0u
- K116: renamed from K16; footprint Cutie Club:ALPS_SKxx_19.05mm -> cutie-lib-alps:Alps_SKxx_19.05mm_1.0u
- K117: renamed from K17; footprint Cutie Club:ALPS_SKxx_19.05mm -> cutie-lib-alps:Alps_SKxx_19.05mm_1.0u
- K118: renamed from K18; footprint Cutie Club:ALPS_SKxx_19.05mm -> cutie-lib-alps:Alps_SKxx_19.05mm_1.0u
- K119: renamed from K19; footprint Cutie Club:ALPS_SKxx_19.05mm -> cutie-lib-alps:Alps_SKxx_19.05mm_1.0u
- K120: renamed from K20; footprint Cutie Club:ALPS_SKxx_19.05mm -> cutie-lib-alps:Alps_SKxx_19.05mm_1.0u
- K121: renamed from K21; footprint Cutie Club:ALPS_SKxx_19.05mm -> cutie-lib-alps:Alps_SKxx_19.05mm_1.0u
- K122: renamed from K22; footprint Cutie Club:ALPS_SKxx_19.05mm -> cutie-lib-alps:Alps_SKxx_19.05mm_1.0u
- K123: renamed from K23; footprint Cutie Club:ALPS_SKxx_19.05mm -> cutie-lib-alps:Alps_SKxx_19.05mm_1.0u
- K124: renamed from K24; footprint Cutie Club:ALPS_SKxx_19.05mm -> cutie-lib-alps:Alps_SKxx_19.05mm_1.0u
- K125: renamed from K25; footprint Cutie Club:ALPS_SKxx_19.05mm -> cutie-lib-alps:Alps_SKxx_19.05mm_1.0u
- K126: renamed from K26; footprint Cutie Club:ALPS_SKxx_19.05mm -> cutie-lib-alps:Alps_SKxx_19.05mm_1.0u
- K127: renamed from K27; footprint Cutie Club:ALPS_SKxx_19.05mm -> cutie-lib-alps:Alps_SKxx_19.05mm_1.0u
- K128: renamed from K28; footprint Cutie Club:ALPS_SKxx_19.05mm -> cutie-lib-alps:Alps_SKxx_19.05mm_1.0u
- K129: renamed from K29; footprint Cutie Club:ALPS_SKxx_19.05mm -> cutie-lib-alps:Alps_SKxx_19.05mm_1.0u
- K130: renamed from K30; footprint Cutie Club:ALPS_SKCLF_19.05mm -> cutie-lib-alps:Alps_SKxx_LED_19.05mm_1.0u
- K131: renamed from K31; footprint Cutie Club:ALPS_SKxx_19.05mm -> cutie-lib-alps:Alps_SKxx_19.05mm_1.0u
- K132: renamed from K32; footprint Cutie Club:ALPS_SKxx_19.05mm -> cutie-lib-alps:Alps_SKxx_19.05mm_1.0u
- K133: renamed from K33; footprint Cutie Club:ALPS_SKxx_19.05mm -> cutie-lib-alps:Alps_SKxx_19.05mm_1.0u
- K134: renamed from K34; footprint Cutie Club:ALPS_SKxx_19.05mm -> cutie-lib-alps:Alps_SKxx_19.05mm_1.0u
- K135: renamed from K35; footprint Cutie Club:ALPS_SKxx_19.05mm -> cutie-lib-alps:Alps_SKxx_19.05mm_1.0u
- K136: renamed from K36; footprint Cutie Club:ALPS_SKxx_19.05mm -> cutie-lib-alps:Alps_SKxx_19.05mm_1.0u
- K137: renamed from K37; footprint Cutie Club:ALPS_SKxx_19.05mm -> cutie-lib-alps:Alps_SKxx_19.05mm_1.0u
- K138: renamed from K38; footprint Cutie Club:ALPS_SKxx_19.05mm -> cutie-lib-alps:Alps_SKxx_19.05mm_1.0u
- K139: renamed from K39; footprint Cutie Club:ALPS_SKxx_19.05mm -> cutie-lib-alps:Alps_SKxx_19.05mm_1.0u
- K140: renamed from K40; footprint Cutie Club:ALPS_SKxx_19.05mm -> cutie-lib-alps:Alps_SKxx_19.05mm_1.0u
- K141: renamed from K41; footprint Cutie Club:ALPS_SKxx_19.05mm -> cutie-lib-alps:Alps_SKxx_19.05mm_1.0u
- K142: renamed from K42; footprint Cutie Club:ALPS_SKxx_19.05mm -> cutie-lib-alps:Alps_SKxx_19.05mm_1.0u
- K143: renamed from K43; footprint Cutie Club:ALPS_SKxx_19.05mm -> cutie-lib-alps:Alps_SKxx_19.05mm_1.0u
- K144: renamed from K44; footprint Cutie Club:ALPS_SKxx_19.05mm -> cutie-lib-alps:Alps_SKxx_19.05mm_1.0u
- K146: renamed from K46; footprint Cutie Club:ALPS_SKxx_19.05mm -> cutie-lib-alps:Alps_SKxx_19.05mm_1.0u
- K147: renamed from K47; footprint Cutie Club:ALPS_SKxx_19.05mm -> cutie-lib-alps:Alps_SKxx_19.05mm_1.0u
- K148: renamed from K48; footprint Cutie Club:ALPS_SKxx_19.05mm -> cutie-lib-alps:Alps_SKxx_19.05mm_1.0u
- K149: renamed from K49; footprint Cutie Club:ALPS_SKxx_19.05mm -> cutie-lib-alps:Alps_SKxx_19.05mm_1.0u
- K150: renamed from K50; footprint Cutie Club:ALPS_SKxx_19.05mm -> cutie-lib-alps:Alps_SKxx_19.05mm_1.0u
- K151: renamed from K51; footprint Cutie Club:ALPS_SKxx_19.05mm -> cutie-lib-alps:Alps_SKxx_19.05mm_1.0u
- K152: renamed from K52; footprint Cutie Club:ALPS_SKxx_19.05mm -> cutie-lib-alps:Alps_SKxx_19.05mm_1.0u
- K153: renamed from K53; footprint Cutie Club:ALPS_SKxx_19.05mm -> cutie-lib-alps:Alps_SKxx_19.05mm_1.0u
- K154: renamed from K54; footprint Cutie Club:ALPS_SKxx_19.05mm -> cutie-lib-alps:Alps_SKxx_19.05mm_1.0u
- K155: renamed from K55; footprint Cutie Club:ALPS_SKxx_19.05mm -> cutie-lib-alps:Alps_SKxx_19.05mm_1.0u
- K156: renamed from K56-2; footprint Cutie Club:ALPS_SKxx_19.05mm -> cutie-lib-alps:Alps_SKxx_19.05mm_1.0u
- K157: renamed from K57; footprint Cutie Club:ALPS_SKxx_19.05mm -> cutie-lib-alps:Alps_SKxx_19.05mm_1.0u
- K158: renamed from K58; footprint Cutie Club:ALPS_SKxx_19.05mm -> cutie-lib-alps:Alps_SKxx_19.05mm_1.0u
- K160: renamed from K60; footprint Cutie Club:ALPS_SKxx_19.05mm -> cutie-lib-alps:Alps_SKxx_19.05mm_1.0u
- K161: renamed from K61; footprint Cutie Club:ALPS_SKxx_19.05mm -> cutie-lib-alps:Alps_SKxx_19.05mm_1.0u
- K162: renamed from K62; footprint Cutie Club:ALPS_SKxx_19.05mm -> cutie-lib-alps:Alps_SKxx_19.05mm_1.0u
- K163: renamed from K63; footprint Cutie Club:ALPS_SKxx_19.05mm -> cutie-lib-alps:Alps_SKxx_19.05mm_1.0u
- K164: renamed from K64; footprint Cutie Club:ALPS_SKxx_19.05mm -> cutie-lib-alps:Alps_SKxx_19.05mm_1.0u
- K165: renamed from K65; footprint Cutie Club:ALPS_SKxx_19.05mm -> cutie-lib-alps:Alps_SKxx_19.05mm_1.0u
- K166: renamed from K66; footprint Cutie Club:ALPS_SKxx_19.05mm -> cutie-lib-alps:Alps_SKxx_19.05mm_1.0u
- K167: renamed from K67; footprint Cutie Club:ALPS_SKxx_19.05mm -> cutie-lib-alps:Alps_SKxx_19.05mm_1.0u
- R102: renamed from R2; value 5.1k -> 1.5k
- R104: renamed from R4; value 10k -> 5.1k
- moved R102 53.5 mm to (335.5, 100.8), turned to 180 degrees
- moved R104 47.7 mm to (328.2, 47.8), turned to -90 degrees
- moved D116 37.0 mm to (300.0, 73.8), turned to -90 degrees
- moved C108 30.0 mm to (329.2, 83.0), turned to 180 degrees
- moved SW101 13.3 mm to (340.5, 100.5)
- moved C105 7.87 mm to (332.0, 100.5), turned to 0 degrees
- moved C107 4.39 mm to (333.2, 92.8), turned to 90 degrees
- moved C110 4.29 mm to (321.8, 54.0), turned to -90 degrees
- moved C103 0.24 mm to (329.2, 81.0)
- renumbered C1 to C101, C2 to C102, C3 to C103, C4 to C104, F1 to F101, J1 to J101, SW1 to SW101, U1 to U101, U2 to U102, U3 to U103
Connections:
- C105 pad 1: VDD -> GND
- C105 pad 2: GND -> BOOT0
- C107 pad 1: RESET -> VDD
- C108 pad 1: +5V -> VDD
- C110 pad 1: Net-(C10-Pad1) -> +5V
- D116 pad 1: ROW0 -> Net-(D116-Pad1)
- D116 pad 2: Net-(D16-Pad2) -> Net-(D116-Pad2)
- J101 pad A8: Net-(J1-PadA8) -> unconnected-(J101-PadA8)
- J101 pad B5: Net-(J1-PadB5) -> Net-(J101-PadB5)
- J101 pad B8: Net-(J1-PadB8) -> unconnected-(J101-PadB8)
- K101 pad 1: Net-(D2-Pad2) -> COL0
- K101 pad 2: COL0 -> Net-(D102-Pad1)
- K102 pad 1: Net-(D3-Pad2) -> COL1
- K102 pad 2: COL1 -> Net-(D102-Pad2)
- K103 pad 1: Net-(D4-Pad2) -> COL2
- K103 pad 2: COL2 -> Net-(D103-Pad1)
- K104 pad 1: Net-(D5-Pad2) -> COL3
- K104 pad 2: COL3 -> Net-(D103-Pad2)
- K105 pad 1: Net-(D6-Pad2) -> COL4
- K105 pad 2: COL4 -> Net-(D104-Pad1)
- K106 pad 1: Net-(D7-Pad2) -> COL5
- K106 pad 2: COL5 -> Net-(D104-Pad2)
- K107 pad 1: Net-(D8-Pad2) -> COL6
- K107 pad 2: COL6 -> Net-(D105-Pad1)
- K108 pad 1: Net-(D9-Pad2) -> COL7
- K108 pad 2: COL7 -> Net-(D105-Pad2)
- K109 pad 1: Net-(D10-Pad2) -> COL8
- K109 pad 2: COL8 -> Net-(D106-Pad1)
- K110 pad 1: Net-(D11-Pad2) -> COL9
- K110 pad 2: COL9 -> Net-(D106-Pad2)
- K111 pad 1: Net-(D12-Pad2) -> COL10
- K111 pad 2: COL10 -> Net-(D107-Pad1)
- K112 pad 1: Net-(D13-Pad2) -> COL11
- K112 pad 2: COL11 -> Net-(D107-Pad2)
- K113 pad 1: Net-(D14-Pad2) -> COL12
- K113 pad 2: COL12 -> Net-(D108-Pad1)
- K114 pad 1: Net-(D15-Pad2) -> COL13
- K114 pad 2: COL13 -> Net-(D108-Pad2)
- K115 pad 2: Net-(D16-Pad2) -> Net-(D109-Pad2)
- K116 pad 1: Net-(D17-Pad2) -> COL0
- K116 pad 2: COL0 -> Net-(D110-Pad1)
- K117 pad 1: Net-(D18-Pad2) -> COL2
- K117 pad 2: COL2 -> Net-(D110-Pad2)
- K118 pad 1: Net-(D19-Pad2) -> COL3
- K118 pad 2: COL3 -> Net-(D111-Pad1)
- K119 pad 1: Net-(D20-Pad2) -> COL4
- K119 pad 2: COL4 -> Net-(D111-Pad2)
- K120 pad 1: Net-(D21-Pad2) -> COL5
- K120 pad 2: COL5 -> Net-(D112-Pad1)
- K121 pad 1: Net-(D22-Pad2) -> COL6
- K121 pad 2: COL6 -> Net-(D112-Pad2)
- K122 pad 1: Net-(D23-Pad2) -> COL7
- K122 pad 2: COL7 -> Net-(D113-Pad1)
- K123 pad 1: Net-(D24-Pad2) -> COL8
- K123 pad 2: COL8 -> Net-(D113-Pad2)
- K124 pad 1: Net-(D25-Pad2) -> COL9
- K124 pad 2: COL9 -> Net-(D114-Pad1)
- K125 pad 1: Net-(D26-Pad2) -> COL10
- K125 pad 2: COL10 -> Net-(D114-Pad2)
- K126 pad 1: Net-(D27-Pad2) -> COL11
- K126 pad 2: COL11 -> Net-(D115-Pad1)
- K127 pad 1: Net-(D28-Pad2) -> COL12
- K127 pad 2: COL12 -> Net-(D115-Pad2)
- K128 pad 1: Net-(D29-Pad2) -> COL13
- K128 pad 2: COL13 -> Net-(D116-Pad1)
- K129 pad 1: COL14 -> Net-(D116-Pad2)
- K129 pad 2: Net-(D30-Pad2) -> COL14
- K130 pad 1: Net-(D31-Pad2) -> COL0
- K130 pad 2: COL0 -> Net-(D117-Pad1)
- K131 pad 1: Net-(D32-Pad2) -> COL2
- K131 pad 2: COL2 -> Net-(D117-Pad2)
- K132 pad 1: Net-(D33-Pad2) -> COL3
- K132 pad 2: COL3 -> Net-(K132-Pad2)
- K133 pad 1: Net-(D34-Pad2) -> COL4
- K133 pad 2: COL4 -> Net-(K133-Pad2)
- K134 pad 1: Net-(D35-Pad2) -> COL5
- K134 pad 2: COL5 -> Net-(D119-Pad1)
- K135 pad 1: Net-(D36-Pad2) -> COL6
- K135 pad 2: COL6 -> Net-(D119-Pad2)
- K136 pad 1: Net-(D37-Pad2) -> COL7
- K136 pad 2: COL7 -> Net-(D120-Pad1)
- K137 pad 1: Net-(D38-Pad2) -> COL8
- K137 pad 2: COL8 -> Net-(D120-Pad2)
- K138 pad 1: Net-(D39-Pad2) -> COL9
- K138 pad 2: COL9 -> Net-(D121-Pad1)
- K139 pad 1: Net-(D40-Pad2) -> COL10
- K139 pad 2: COL10 -> Net-(D121-Pad2)
- K140 pad 1: Net-(D41-Pad2) -> COL11
- K140 pad 2: COL11 -> Net-(D122-Pad1)
- K141 pad 1: Net-(D42-Pad2) -> COL12
- K141 pad 2: COL12 -> Net-(D122-Pad2)
- K142 pad 1: Net-(D43-Pad2) -> COL13
- K142 pad 2: COL13 -> Net-(K142-Pad2)
- K143 pad 1: Net-(D44-Pad2) -> COL14
- K143 pad 2: COL14 -> Net-(K143-Pad2)
- K144 pad 1: Net-(D45-Pad2) -> COL0
- K144 pad 2: COL0 -> Net-(D124-Pad1)
- K146 pad 1: Net-(D47-Pad2) -> COL2
- K146 pad 2: COL2 -> Net-(D125-Pad1)
- K147 pad 1: Net-(D48-Pad2) -> COL3
- K147 pad 2: COL3 -> Net-(D125-Pad2)
- K148 pad 1: Net-(D49-Pad2) -> COL4
- K148 pad 2: COL4 -> Net-(D126-Pad1)
- K149 pad 1: Net-(D50-Pad2) -> COL5
- K149 pad 2: COL5 -> Net-(D126-Pad2)
- K150 pad 1: Net-(D51-Pad2) -> COL6
- K150 pad 2: COL6 -> Net-(D127-Pad1)
- K151 pad 1: Net-(D52-Pad2) -> COL7
- K151 pad 2: COL7 -> Net-(D127-Pad2)
- K152 pad 1: Net-(D53-Pad2) -> COL8
- K152 pad 2: COL8 -> Net-(D128-Pad1)
- K153 pad 1: Net-(D54-Pad2) -> COL9
- K153 pad 2: COL9 -> Net-(D128-Pad2)
- K154 pad 1: Net-(D55-Pad2) -> COL10
- K154 pad 2: COL10 -> Net-(D129-Pad1)
- K155 pad 1: Net-(D56-Pad2) -> COL11
- K155 pad 2: COL11 -> Net-(D129-Pad2)
- K156 pad 1: Net-(D57-Pad2) -> COL12
- K156 pad 2: COL12 -> Net-(D130-Pad1)
- K157 pad 1: Net-(D58-Pad2) -> COL13
- K157 pad 2: COL13 -> Net-(D130-Pad2)
- K158 pad 1: Net-(D59-Pad2) -> COL14
- K158 pad 2: COL14 -> Net-(D131-Pad1)
- K160 pad 1: COL1 -> Net-(D132-Pad2)
- K160 pad 2: Net-(D61-Pad2) -> COL1
- K161 pad 1: COL2 -> Net-(D133-Pad1)
- K161 pad 2: Net-(D62-Pad2) -> COL2
- K162 pad 1: COL6 -> Net-(D133-Pad2)
- K162 pad 2: Net-(D63-Pad2) -> COL6
- K163 pad 1: Net-(D64-Pad2) -> COL10
- K163 pad 2: COL10 -> Net-(D134-Pad1)
- K164 pad 1: Net-(D65-Pad2) -> COL11
- K164 pad 2: COL11 -> Net-(D134-Pad2)
- K165 pad 1: Net-(D66-Pad2) -> COL12
- K165 pad 2: COL12 -> Net-(D135-Pad1)
- K166 pad 1: Net-(D67-Pad2) -> COL13
- K166 pad 2: COL13 -> Net-(D135-Pad2)
- K167 pad 1: Net-(D68-Pad2) -> COL14
- K167 pad 2: COL14 -> Net-(D136-Pad2)
- R102 pad 1: Net-(J1-PadB5) -> Net-(D101-Pad2)
- R102 pad 2: GND -> Net-(Q101-Pad1)
- R104 pad 1: Net-(R4-Pad1) -> Net-(J101-PadB5)
- R104 pad 2: BOOT0 -> GND
- SW101 pad 1: RESET -> VDD
- SW101 pad 2: GND -> Net-(D101-Pad2)
- U101 pad 2: Net-(U1-Pad2) -> unconnected-(U101-Pad2)
- U101 pad 27: Net-(U1-Pad27) -> unconnected-(U101-Pad27)
- U101 pad 28: Net-(U1-Pad28) -> unconnected-(U101-Pad28)
- U101 pad 29: Net-(U1-Pad29) -> unconnected-(U101-Pad29)
- U101 pad 3: Net-(U1-Pad3) -> unconnected-(U101-Pad3)
- U101 pad 30: Net-(U1-Pad30) -> unconnected-(U101-Pad30)
- U101 pad 31: Net-(U1-Pad31) -> unconnected-(U101-Pad31)
- U101 pad 34: Net-(U1-Pad34) -> unconnected-(U101-Pad34)
- U101 pad 39: Net-(U1-Pad39) -> unconnected-(U101-Pad39)
- U101 pad 4: Net-(U1-Pad4) -> unconnected-(U101-Pad4)
- U101 pad 42: Net-(U1-Pad42) -> unconnected-(U101-Pad42)
- U101 pad 43: Net-(U1-Pad43) -> unconnected-(U101-Pad43)
- U101 pad 45: Net-(U1-Pad45) -> unconnected-(U101-Pad45)
- U101 pad 46: Net-(U1-Pad46) -> unconnected-(U101-Pad46)
- U102 pad 4: Net-(C10-Pad1) -> Net-(C111-Pad1)
Routing:
- net Net-(D133-Pad2): track 0.00 -> 77.4 mm
- net Net-(D116-Pad2): track 0.00 -> 37.9 mm
- net Net-(D130-Pad1): track 0.00 -> 29.4 mm
- net Net-(D57-Pad2): track 23.1 -> 0.00 mm
- net Net-(D117-Pad2): track 0.00 -> 19.1 mm
- net Net-(D132-Pad2): track 0.00 -> 17.3 mm
- net Net-(D134-Pad1): track 0.00 -> 17.1 mm
- net Net-(D110-Pad2): track 0.00 -> 16.8 mm
- net Net-(K143-Pad2): track 0.00 -> 16.5 mm, vias 0 -> 1
- net Net-(D108-Pad2): track 0.00 -> 16.5 mm
- net Net-(D124-Pad2): track 0.00 -> 14.4 mm
- net Net-(D15-Pad2): track 14.1 -> 0.00 mm
- net Net-(D135-Pad1): track 0.00 -> 12.3 mm
- net Net-(D121-Pad2): track 0.00 -> 12.0 mm
- net Net-(D120-Pad2): track 0.00 -> 12.0 mm
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Other:
- board text added: "-+"
- board text added: "Borsdorf CC BY-SA 4.0 cutieclub.cc 2023"
