File: borsdorf.kicad_sch (KiCad schematic)
At the start: 158 parts

Commit message: Update files to v2/extras revision
Parts:
- removed D10, D11, D12, D13, D14, D15, D16, D17, D18, D19, D2, D20, D21, D22, D23, D24, D25, D26, D27, D28, D29, D3, D30, D31, D32, D33, D34, D35, D36, D37, D38, D39, D4, D40, D41, D42, D43, D44, D45, D46, D47, D48, D49, D5, D50, D51, D52, D53, D54, D55, D56, D57, D58, D59, D6, D60, D61, D62, D63, D64, D65, D66, D67, D68, D7, D8, D9: (no value), symbol borsdorf-rescue:D_Small_ALT-Device
- removed K31, K58: (no value), symbol Switch:SW_SPST
- removed SW2: (no value), symbol Switch:SW_SPDT
- added D101: 1N4148, Diode_SMD:D_SOD-323, symbol Device:D_Small_Filled
- added D102, D103, D104, D105, D106, D107, D108, D109, D110, D111, D112, D113, D114, D115, D116, D117, D118, D119, D120, D121, D122, D123, D124, D125, D126, D127, D128, D129, D130, D131, D132, D133, D134, D135, D136: BAV70, Package_TO_SOT_SMD:SOT-23, symbol Diode:BAV70
- added K143, K145: KEYSW, cutie-lib-alps:Alps_SKxx_19.05mm_1.0u, symbol Switch:SW_SPST
- added Q101: MBT2222A, Package_TO_SOT_SMD:SOT-23-3, symbol Device:Q_NPN_BCE
- added R102: 1.5k, Resistor_SMD:R_0805_2012Metric, symbol Device:R_Small
- C101: renamed from C1; value (none) -> 100nF; footprint (none) -> Capacitor_SMD:C_0805_2012Metric
- C102: renamed from C2; value (none) -> 1uF; footprint (none) -> Capacitor_SMD:C_0805_2012Metric
- C103: renamed from C3; value (none) -> 4.7uF; footprint (none) -> Capacitor_SMD:C_0805_2012Metric
- C104: renamed from C4; value (none) -> 4.7uF; footprint (none) -> Capacitor_SMD:C_0805_2012Metric
- C105: renamed from C7; value (none) -> 10uF; footprint (none) -> Capacitor_SMD:C_0805_2012Metric
- C106: renamed from C5; value (none) -> 100nF; footprint (none) -> Capacitor_SMD:C_0805_2012Metric
- C107: renamed from C6; value (none) -> 10nF; footprint (none) -> Capacitor_SMD:C_0805_2012Metric
- C108: renamed from C12; value (none) -> 100nF; footprint (none) -> Capacitor_SMD:C_0805_2012Metric
- C109: renamed from C8; value (none) -> 1uF; footprint (none) -> Capacitor_SMD:C_0805_2012Metric
- C110: renamed from C9; value (none) -> 100nF; footprint (none) -> Capacitor_SMD:C_0805_2012Metric
- C111: renamed from C10; value (none) -> 10nF; footprint (none) -> Capacitor_SMD:C_0805_2012Metric
- C112: renamed from C11; value (none) -> 2.2uF; footprint (none) -> Capacitor_SMD:C_0805_2012Metric
- F101: renamed from F1; value (none) -> PTTC; footprint (none) -> Fuse:Fuse_0805_2012Metric
- J101: renamed from J1; value (none) -> USB2.0-USB-C; footprint (none) -> Connector_USB:USB_C_Receptacle_HRO_TYPE-C-31-M-12
- K101: renamed from K5; value (none) -> KEYSW; footprint (none) -> cutie-lib-alps:Alps_SKxx_19.05mm_1.0u
- K102: renamed from K4; value (none) -> KEYSW; footprint (none) -> cutie-lib-alps:Alps_SKxx_19.05mm_1.0u
- K103: renamed from K3; value (none) -> KEYSW; footprint (none) -> cutie-lib-alps:Alps_SKxx_19.05mm_1.0u
- K104: renamed from K2; value (none) -> KEYSW; footprint (none) -> cutie-lib-alps:Alps_SKxx_19.05mm_1.0u
- K105: renamed from K1; value (none) -> KEYSW; footprint (none) -> cutie-lib-alps:Alps_SKxx_19.05mm_1.0u
- K106: renamed from K6; value (none) -> KEYSW; footprint (none) -> cutie-lib-alps:Alps_SKxx_19.05mm_1.0u
- K107: renamed from K7; value (none) -> KEYSW; footprint (none) -> cutie-lib-alps:Alps_SKxx_19.05mm_1.0u
- K108: renamed from K8; value (none) -> KEYSW; footprint (none) -> cutie-lib-alps:Alps_SKxx_19.05mm_1.0u
- K109: renamed from K9; value (none) -> KEYSW; footprint (none) -> cutie-lib-alps:Alps_SKxx_19.05mm_1.0u
- K110: renamed from K10; value (none) -> KEYSW; footprint (none) -> cutie-lib-alps:Alps_SKxx_19.05mm_1.0u
- K111: renamed from K11; value (none) -> KEYSW; footprint (none) -> cutie-lib-alps:Alps_SKxx_19.05mm_1.0u
- K112: renamed from K12; value (none) -> KEYSW; footprint (none) -> cutie-lib-alps:Alps_SKxx_19.05mm_1.0u
- K113: renamed from K13; value (none) -> KEYSW; footprint (none) -> cutie-lib-alps:Alps_SKxx_19.05mm_1.0u
- K114: renamed from K14; value (none) -> KEYSW; footprint (none) -> cutie-lib-alps:Alps_SKxx_19.05mm_1.0u
- K115: renamed from K15; value (none) -> KEYSW; footprint (none) -> cutie-lib-alps:Alps_SKxx_19.05mm_1.0u
- K116: renamed from K16; value (none) -> KEYSW; footprint (none) -> cutie-lib-alps:Alps_SKxx_19.05mm_1.0u
- K117: renamed from K17; value (none) -> KEYSW; footprint (none) -> cutie-lib-alps:Alps_SKxx_19.05mm_1.0u
- K118: renamed from K18; value (none) -> KEYSW; footprint (none) -> cutie-lib-alps:Alps_SKxx_19.05mm_1.0u
- K119: renamed from K19; value (none) -> KEYSW; footprint (none) -> cutie-lib-alps:Alps_SKxx_19.05mm_1.0u
- K120: renamed from K20; value (none) -> KEYSW; footprint (none) -> cutie-lib-alps:Alps_SKxx_19.05mm_1.0u
- K121: renamed from K21; value (none) -> KEYSW; footprint (none) -> cutie-lib-alps:Alps_SKxx_19.05mm_1.0u
- K122: renamed from K22; value (none) -> KEYSW; footprint (none) -> cutie-lib-alps:Alps_SKxx_19.05mm_1.0u
- K123: renamed from K23; value (none) -> KEYSW; footprint (none) -> cutie-lib-alps:Alps_SKxx_19.05mm_1.0u
- K124: renamed from K24; value (none) -> KEYSW; footprint (none) -> cutie-lib-alps:Alps_SKxx_19.05mm_1.0u
- K125: renamed from K25; value (none) -> KEYSW; footprint (none) -> cutie-lib-alps:Alps_SKxx_19.05mm_1.0u
- K126: renamed from K26; value (none) -> KEYSW; footprint (none) -> cutie-lib-alps:Alps_SKxx_19.05mm_1.0u
- K127: renamed from K27; value (none) -> KEYSW; footprint (none) -> cutie-lib-alps:Alps_SKxx_19.05mm_1.0u
- K128: renamed from K28; value (none) -> KEYSW; footprint (none) -> cutie-lib-alps:Alps_SKxx_19.05mm_1.0u
- K129: renamed from K29; value (none) -> KEYSW; footprint (none) -> cutie-lib-alps:Alps_SKxx_19.05mm_1.0u
- K130: renamed from K30; value (none) -> KEYSW; footprint (none) -> cutie-lib-alps:Alps_SKxx_LED_19.05mm_1.0u
- K131: renamed from K32; value (none) -> KEYSW; footprint (none) -> cutie-lib-alps:Alps_SKxx_19.05mm_1.0u
- K132: renamed from K33; value (none) -> KEYSW; footprint (none) -> cutie-lib-alps:Alps_SKxx_19.05mm_1.0u
- K133: renamed from K34; value (none) -> KEYSW; footprint (none) -> cutie-lib-alps:Alps_SKxx_19.05mm_1.0u
- K134: renamed from K35; value (none) -> KEYSW; footprint (none) -> cutie-lib-alps:Alps_SKxx_19.05mm_1.0u
- K135: renamed from K36; value (none) -> KEYSW; footprint (none) -> cutie-lib-alps:Alps_SKxx_19.05mm_1.0u
- K136: renamed from K37; value (none) -> KEYSW; footprint (none) -> cutie-lib-alps:Alps_SKxx_19.05mm_1.0u
- K137: renamed from K38; value (none) -> KEYSW; footprint (none) -> cutie-lib-alps:Alps_SKxx_19.05mm_1.0u
- K138: renamed from K39; value (none) -> KEYSW; footprint (none) -> cutie-lib-alps:Alps_SKxx_19.05mm_1.0u
- K139: renamed from K40; value (none) -> KEYSW; footprint (none) -> cutie-lib-alps:Alps_SKxx_19.05mm_1.0u
- K140: renamed from K41; value (none) -> KEYSW; footprint (none) -> cutie-lib-alps:Alps_SKxx_19.05mm_1.0u
- K141: renamed from K42; value (none) -> KEYSW; footprint (none) -> cutie-lib-alps:Alps_SKxx_19.05mm_1.0u
- K142: renamed from K43; value (none) -> KEYSW; footprint (none) -> cutie-lib-alps:Alps_SKxx_19.05mm_1.0u
- K144: renamed from K44; value (none) -> KEYSW; footprint (none) -> cutie-lib-alps:Alps_SKxx_19.05mm_1.0u
- K146: renamed from K45; value (none) -> KEYSW; footprint (none) -> cutie-lib-alps:Alps_SKxx_19.05mm_1.0u
- K147: renamed from K46; value (none) -> KEYSW; footprint (none) -> cutie-lib-alps:Alps_SKxx_19.05mm_1.0u
- K148: renamed from K47; value (none) -> KEYSW; footprint (none) -> cutie-lib-alps:Alps_SKxx_19.05mm_1.0u
- K149: renamed from K48; value (none) -> KEYSW; footprint (none) -> cutie-lib-alps:Alps_SKxx_19.05mm_1.0u
- K150: renamed from K49; value (none) -> KEYSW; footprint (none) -> cutie-lib-alps:Alps_SKxx_19.05mm_1.0u
- K151: renamed from K50; value (none) -> KEYSW; footprint (none) -> cutie-lib-alps:Alps_SKxx_19.05mm_1.0u
- K152: renamed from K51; value (none) -> KEYSW; footprint (none) -> cutie-lib-alps:Alps_SKxx_19.05mm_1.0u
- K153: renamed from K52; value (none) -> KEYSW; footprint (none) -> cutie-lib-alps:Alps_SKxx_19.05mm_1.0u
- K154: renamed from K53; value (none) -> KEYSW; footprint (none) -> cutie-lib-alps:Alps_SKxx_19.05mm_1.0u
- K155: renamed from K54; value (none) -> KEYSW; footprint (none) -> cutie-lib-alps:Alps_SKxx_19.05mm_1.0u
- K156: renamed from K55; value (none) -> KEYSW; footprint (none) -> cutie-lib-alps:Alps_SKxx_19.05mm_1.0u
- K157: renamed from K56; value (none) -> KEYSW; footprint (none) -> cutie-lib-alps:Alps_SKxx_19.05mm_1.0u
- K1571: renamed from K56-2; value (none) -> KEYSW; footprint (none) -> cutie-lib-alps:Alps_SKxx_19.05mm_1.0u
- K158: renamed from K57; value (none) -> KEYSW; footprint (none) -> cutie-lib-alps:Alps_SKxx_19.05mm_1.0u
- K159: renamed from K59; value (none) -> KEYSW; footprint (none) -> cutie-lib-alps:Alps_SKxx_19.05mm_1.0u
- K160: renamed from K60; value (none) -> KEYSW; footprint (none) -> cutie-lib-alps:Alps_SKxx_19.05mm_1.0u
- K161: renamed from K61; value (none) -> KEYSW; footprint (none) -> cutie-lib-alps:Alps_SKxx_19.05mm_1.0u
- K162: renamed from K62; value (none) -> KEYSW; footprint (none) -> cutie-lib-alps:Alps_SKxx_19.05mm_1.0u
- K163: renamed from K63; value (none) -> KEYSW; footprint (none) -> cutie-lib-alps:Alps_SKxx_19.05mm_1.0u
- K164: renamed from K64; value (none) -> KEYSW; footprint (none) -> cutie-lib-alps:Alps_SKxx_19.05mm_1.0u
- K165: renamed from K65; value (none) -> KEYSW; footprint (none) -> cutie-lib-alps:Alps_SKxx_19.05mm_1.0u
- K166: renamed from K66; value (none) -> KEYSW; footprint (none) -> cutie-lib-alps:Alps_SKxx_19.05mm_1.0u
- K167: renamed from K67; value (none) -> KEYSW; footprint (none) -> cutie-lib-alps:Alps_SKxx_19.05mm_1.0u
- R101: renamed from R3; value (none) -> 5.1k; footprint (none) -> Resistor_SMD:R_0805_2012Metric
- R103: renamed from R4; value (none) -> 30k; footprint (none) -> Resistor_SMD:R_0805_2012Metric
- R104: renamed from R2; value (none) -> 5.1k; footprint (none) -> Resistor_SMD:R_0805_2012Metric
- R105: renamed from R1; value (none) -> R_Small; footprint (none) -> Resistor_SMD:R_0805_2012Metric
- SW101: renamed from SW1; value (none) -> ALPS SKRK; footprint (none) -> Cutie Club:ALPS_SKRK; symbol borsdorf-rescue:Switch-Cutie_Club -> Switch:SW_SPST
- U101: renamed from U1; value (none) -> STM32F072CBTx; footprint (none) -> Package_QFP:LQFP-48_7x7mm_P0.5mm
- U102: renamed from U2; value (none) -> LP2985-3.3; footprint (none) -> Package_TO_SOT_SMD:SOT-23-5
- U103: renamed from U3; value (none) -> USBLC6-2P6; footprint (none) -> Package_TO_SOT_SMD:SOT-23-6
Connections:
- net BOOT0: now also C105.2, R103.1, D101.1 (K); no longer R103.2
- net COL0: now also K101.1 (A), K116.1 (A), K130.1, K144.1 (A), K159.2 (B); no longer K105.2 (B), K116.2 (B), K130.2, K144.2 (B), K159.1 (A)
- net COL1: now also K102.1 (A), K160.2 (B), K145.1 (A); no longer K104.2 (B), K146.2 (B), K160.1 (A)
- net COL10: now also K111.1 (A), K125.1 (A), K139.1 (A), K154.1 (A), K163.1 (A); no longer K111.2 (B), K125.2 (B), K138.2 (B), K155.2 (B), K163.2 (B)
- net COL11: now also K112.1 (A), K126.1 (A), K140.1 (A), K155.1 (A), K164.1 (A); no longer K112.2 (B), K126.2 (B), K139.2 (B), K156.2 (B), K164.2 (B)
- net COL12: now also K113.1 (A), K127.1 (A), K141.1 (A), K156.1 (A), K1571.1 (A), K165.1 (A); no longer K113.2 (B), K127.2 (B), K140.2 (B), K157.2 (B), K1571.2 (B), K165.2 (B)
- net COL13: now also K114.1 (A), K128.1 (A), K142.1 (A), K157.1 (A), K166.1 (A); no longer K114.2 (B), K128.2 (B), K141.2 (B), K158.2 (B), K166.2 (B)
- net COL14: now also K129.2 (B), K158.1 (A), K167.1 (A), K143.1 (A); no longer K129.1 (A), K142.2 (B), K167.2 (B)
- net COL2: now also K103.1 (A), K117.1 (A), K131.1 (A), K146.1 (A), K161.2 (B); no longer K103.2 (B), K117.2 (B), K147.2 (B), K161.1 (A)
- net COL3: now also K104.1 (A), K118.1 (A), K132.1 (A), K147.1 (A); no longer K102.2 (B), K118.2 (B), K131.2 (B), K148.2 (B)
- net COL4: now also K105.1 (A), K119.1 (A), K133.1 (A), K148.1 (A); no longer K101.2 (B), K119.2 (B), K132.2 (B), K149.2 (B)
- net COL5: now also K106.1 (A), K120.1 (A), K134.1 (A), K149.1 (A); no longer K106.2 (B), K120.2 (B), K133.2 (B), K150.2 (B)
- net COL6: now also K107.1 (A), K121.1 (A), K135.1 (A), K150.1 (A), K162.2 (B); no longer K107.2 (B), K121.2 (B), K134.2 (B), K151.2 (B), K162.1 (A)
- net COL7: now also K108.1 (A), K122.1 (A), K136.1 (A), K151.1 (A); no longer K108.2 (B), K122.2 (B), K135.2 (B), K152.2 (B)
- net COL8: now also K109.1 (A), K123.1 (A), K137.1 (A), K152.1 (A); no longer K109.2 (B), K123.2 (B), K136.2 (B), K153.2 (B)
- net COL9: now also K110.1 (A), K124.1 (A), K138.1 (A), K153.1 (A); no longer K110.2 (B), K124.2 (B), K137.2 (B), K154.2 (B)
- net GND: now also C105.1, R103.2, Q101.3 (E); no longer C105.2, SW101.2
- net RESET: now also Q101.2 (C); no longer C105.1, SW101.1
- net ROW0: now also D102.3 (K), D103.3 (K), D104.3 (K), D105.3 (K), D106.3 (K), D107.3 (K), D108.3 (K), D109.3 (K)
- net ROW1: now also D110.3 (K), D111.3 (K), D112.3 (K), D113.3 (K), D114.3 (K), D115.3 (K), D116.3 (K)
- net ROW2: now also D117.3 (K), D118.3 (K), D119.3 (K), D120.3 (K), D121.3 (K), D122.3 (K), D123.3 (K)
- net ROW3: now also D124.3 (K), D125.3 (K), D126.3 (K), D127.3 (K), D128.3 (K), D129.3 (K), D130.3 (K), D131.3 (K)
- net ROW4: now also D132.3 (K), D133.3 (K), D134.3 (K), D135.3 (K), D136.3 (K)
- net VDD: now also SW101.1 (A)
- net at K115.2 (B): now also D109.2 (A)
- new net: D104.1 (A), K105.2 (B)
- new net: D103.2 (A), K104.2 (B)
- new net: D103.1 (A), K103.2 (B)
- new net: D110.2 (A), K117.2 (B)
- new net: D125.2 (A), K147.2 (B)
- new net: D133.1 (A), K161.1 (A)
- new net: D125.1 (A), K146.2 (B)
- new net: D110.1 (A), K116.2 (B)
- new net: D124.1 (A), K144.2 (B)
- new net: D132.1 (A), K159.1 (A)
- new net: D102.2 (A), K102.2 (B)
- new net: D102.1 (A), K101.2 (B)
- new net: D104.2 (A), K106.2 (B)
- new net: D105.1 (A), K107.2 (B)
- new net: D105.2 (A), K108.2 (B)
- new net: D106.1 (A), K109.2 (B)
- new net: D106.2 (A), K110.2 (B)
- new net: D107.1 (A), K111.2 (B)
- new net: D107.2 (A), K112.2 (B)
- new net: D108.1 (A), K113.2 (B)
- new net: D108.2 (A), K114.2 (B)
- new net: D132.2 (A), K160.1 (A)
- new net: D111.1 (A), K118.2 (B)
- new net: D117.2 (A), K131.2 (B)
- new net: D126.1 (A), K148.2 (B)
- new net: D111.2 (A), K119.2 (B)
- new net: D118.1 (A), K132.2 (B)
- new net: D126.2 (A), K149.2 (B)
- new net: D112.1 (A), K120.2 (B)
- new net: D118.2 (A), K133.2 (B)
- new net: D127.1 (A), K150.2 (B)
- new net: D112.2 (A), K121.2 (B)
- new net: D119.1 (A), K134.2 (B)
- new net: D127.2 (A), K151.2 (B)
- new net: D133.2 (A), K162.1 (A)
- new net: D113.1 (A), K122.2 (B)
- new net: D119.2 (A), K135.2 (B)
- new net: D128.1 (A), K152.2 (B)
- new net: D113.2 (A), K123.2 (B)
- new net: D120.1 (A), K136.2 (B)
- new net: D128.2 (A), K153.2 (B)
- new net: D114.1 (A), K124.2 (B)
- new net: D120.2 (A), K137.2 (B)
- new net: D129.1 (A), K154.2 (B)
- new net: D114.2 (A), K125.2 (B)
- new net: D121.1 (A), K138.2 (B)
- new net: D129.2 (A), K155.2 (B)
- new net: D115.1 (A), K126.2 (B)
- new net: D121.2 (A), K139.2 (B)
- new net: D130.1 (A), K156.2 (B), K1571.2 (B)
- new net: D115.2 (A), K127.2 (B)
- new net: D122.1 (A), K140.2 (B)
- new net: D134.2 (A), K164.2 (B)
- new net: D134.1 (A), K163.2 (B)
- new net: D116.1 (A), K128.2 (B)
- new net: D122.2 (A), K141.2 (B)
- new net: D131.1 (A), K158.2 (B)
- new net: D135.1 (A), K165.2 (B)
- new net: D135.2 (A), K166.2 (B)
- new net: D130.2 (A), K157.2 (B)
- new net: D116.2 (A), K129.1 (A)
- new net: D136.2 (A), K167.2 (B)
- new net: D123.1 (A), K142.2 (B)
- new net: D101.2 (A), R102.1, SW101.2 (B)
- new net: D117.1 (A), K130.2
- new net: D123.2 (A), K143.2 (B)
- new net: Q101.1 (B), R102.2
- new net: D124.2 (A), K145.2 (B)
- no-connect marks 16 -> 18
Other:
- note added: "Switch Matrix"
- note removed: "Switch Matrix - all good"
- moved on the sheet: C105, K101, K102, K103, K104, K105, K106, K107, K108, K109, K110, K111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
